Commit message: added pickable objects

File: src/so101_description/urdf/dual_arm_workcell_gazebo.urdf.xacro (robot description, xacro)
@@ -6,8 +6,11 @@
   can be spawned into Gazebo (mirrors the existing dual_arm_gazebo.urdf.xacro
   pattern).
-  The sole manipulable object pair is the 4-pin plug and its matching
-  4-pocket socket. The earlier single-peg/hole-plate setup (fixture, base
-  plate, peg, parts tray) still exists, just moved out of the active
-  workcell into dual_arm_workcell_peghole_gazebo.urdf.xacro.
+  The socket (4-pocket) is the only assembly object defined here, fixed to
+  the table. Its matching 4-pin plug is a genuine free rigid body instead,
+  spawned separately as models/plug.sdf by workcell_gazebo.launch.py so it
+  can actually be picked up, with its ground-truth pose bridged to ROS 2
+  for later perception evaluation. The earlier single-peg/hole-plate setup
+  (fixture, base plate, peg, parts tray) still exists, just moved out of the
+  active workcell into dual_arm_workcell_peghole_gazebo.urdf.xacro.
   The wrist cameras are mounted physically (mesh + link + joint, via the
   so101_*_arm_camera fragments) but intentionally have no gazebo sensor
@@ -48,7 +51,11 @@
   <xacro:property name="cam_yaw"   value="${-pi/2}"/>
   <!-- ================= ASSEMBLY AREA ================= -->
-  <!-- The only manipulable objects are the 4-pin plug and socket: the
-       single-peg/hole-plate setup now lives separately in
-       dual_arm_workcell_peghole_gazebo.urdf.xacro. -->
+  <!-- Socket is static, fixed to the table. The plug is a separately
+       spawned free body (models/plug.sdf), not part of this URDF, see
+       workcell_gazebo.launch.py. plug_x/plug_y are kept here only so the
+       launch file's spawn position (world frame: x=plug_x, y=plug_y,
+       z=table_top_z, since table_link has no rotation/xy-offset from
+       world) stays next to the property that defines it, for the same
+       spot the plug used to occupy when it was welded to the table. -->
   <xacro:property name="socket_x" value="0.0"/>
   <xacro:property name="socket_y" value="0.08"/>
@@ -282,11 +289,11 @@
     <origin xyz="0 0 0" rpy="${-pi/2} 0 ${-pi/2}"/>
   </joint>
-  <!-- ================= 4-PIN PLUG / SOCKET ================= -->
-  <!-- Socket fixed to the table; plug sits loose nearby, pins up, ready to
-       be picked up and inserted. -->
+  <!-- ================= SOCKET (static) ================= -->
+  <!-- The plug is NOT instantiated here: it's a free rigid body, spawned
+       separately as models/plug.sdf via `ros2 run ros_gz_sim create` in
+       workcell_gazebo.launch.py (at plug_x/plug_y, same spot as before) so
+       it's actually pickable rather than welded to the table. -->
   <xacro:socket name="socket" parent="table_link"
     xyz="${socket_x} ${socket_y} 0" rpy="0 0 0"/>
-  <xacro:plug name="plug" parent="table_link"
-    xyz="${plug_x} ${plug_y} 0" rpy="0 0 0"/>
   <!-- ================= ROS2_CONTROL ================ -->
   <xacro:macro name="position_joint" params="name">

File: src/so101_description/urdf/dual_arm_workcell_peghole.urdf.xacro (robot description, xacro)
@@ -40,5 +40,6 @@
   <xacro:property name="gantry_post_height" value="0.55"/>
   <xacro:property name="gantry_post_x"      value="0.46"/>
-  <xacro:property name="cam_pitch" value="${pi/3}"/>
+  <!-- pitch=85deg: 5deg off straight-down (was 60deg/30deg) -->
+  <xacro:property name="cam_pitch" value="${pi*85/180}"/>
   <xacro:property name="cam_yaw"   value="${-pi/2}"/>
   <!-- ================= ASSEMBLY AREA ================= -->

File: src/so101_description/urdf/dual_arm_workcell_peghole_gazebo.urdf.xacro (robot description, xacro)
@@ -2,8 +2,14 @@
 <!--
   Dual-arm assembly workcell (Gazebo Harmonic variant): same table, arms,
-  overhead camera and assembly objects as dual_arm_workcell.urdf.xacro, plus
-  ros2_control command/state interfaces and the gz_ros2_control plugin so it
-  can be spawned into Gazebo (mirrors the existing dual_arm_gazebo.urdf.xacro
-  pattern).
+  overhead camera and assembly objects as dual_arm_workcell_peghole.urdf.xacro,
+  plus ros2_control command/state interfaces and the gz_ros2_control plugin
+  so it can be spawned into Gazebo (mirrors the existing
+  dual_arm_gazebo.urdf.xacro pattern).
+  The assembly fixture, base plate, socket, and parts tray (with its two
+  decorative spare pegs) are all static, fixed to the table here. The
+  functional peg and 4-pin plug are instead genuine free rigid bodies,
+  spawned separately as models/peg.sdf and models/plug.sdf by
+  workcell_peghole_gazebo.launch.py so they can actually be picked up, with
+  their ground-truth poses bridged to ROS 2 for later perception evaluation.
   The wrist cameras are mounted physically (mesh + link + joint, via the
   so101_*_arm_camera fragments) but intentionally have no gazebo sensor
@@ -40,5 +46,6 @@
   <xacro:property name="gantry_post_height" value="0.55"/>
   <xacro:property name="gantry_post_x"      value="0.46"/>
-  <xacro:property name="cam_pitch" value="${pi/3}"/>
+  <!-- pitch=85deg: 5deg off straight-down (was 60deg/30deg) -->
+  <xacro:property name="cam_pitch" value="${pi*85/180}"/>
   <xacro:property name="cam_yaw"   value="${-pi/2}"/>
   <!-- ================= ASSEMBLY AREA ================= -->
@@ -280,12 +287,17 @@
     <origin xyz="0 0 0" rpy="${-pi/2} 0 ${-pi/2}"/>
   </joint>
-  <!-- ================= ASSEMBLY FIXTURE + BASE PLATE ================= -->
+  <!-- ================= ASSEMBLY FIXTURE + BASE PLATE (static) ================= -->
+  <!-- The peg is NOT instantiated here: it's a free rigid body, spawned
+       separately as models/peg.sdf via `ros2 run ros_gz_sim create` in
+       workcell_peghole_gazebo.launch.py (at the same spot it used to
+       occupy: x = fixture_x + 0.09, y = fixture_y) so it's actually
+       pickable rather than welded to the table. -->
   <xacro:assembly_fixture name="assembly_fixture" parent="table_link"
     xyz="${fixture_x} ${fixture_y} 0" rpy="0 0 0"/>
   <xacro:base_plate_with_hole name="base_plate" parent="assembly_fixture_link"
     xyz="0 0 0.006" rpy="0 0 0"/>
-  <xacro:peg name="assembly_peg" parent="table_link"
-    xyz="${fixture_x + 0.09} ${fixture_y} 0" rpy="0 0 0"/>
   <!-- ================= PARTS TRAY ================= -->
+  <!-- Spare pegs stay fixed/decorative: only the functional peg and plug
+       were asked to become pickable, not every loose part in the scene. -->
   <xacro:parts_tray name="parts_tray" parent="table_link"
     xyz="${tray_x} ${tray_y} 0" rpy="0 0 0"/>
@@ -294,11 +306,9 @@
   <xacro:peg name="spare_peg_2" parent="parts_tray_link"
     xyz="0.02 -0.015 0.013" rpy="0 ${pi/2} ${pi/4}" radius="0.007" length="0.035"/>
-  <!-- ================= 4-PIN PLUG / SOCKET ================= -->
-  <!-- Socket fixed to the table; plug sits loose nearby, pins up, ready to
-       be picked up and inserted. -->
+  <!-- ================= SOCKET (static) ================= -->
+  <!-- The plug is likewise spawned separately as models/plug.sdf, not
+       instantiated here, see workcell_peghole_gazebo.launch.py. -->
   <xacro:socket name="socket" parent="table_link"
     xyz="${socket_x} ${socket_y} 0" rpy="0 0 0"/>
-  <xacro:plug name="plug" parent="table_link"
-    xyz="${plug_x} ${plug_y} 0" rpy="0 0 0"/>
   <!-- ================= ROS2_CONTROL ================ -->
   <xacro:macro name="position_joint" params="name">

Commit message: Assembly with ground position values is tested

File: src/so101_description/urdf/dual_arm_workcell_gazebo.urdf.xacro (robot description, xacro)
@@ -22,6 +22,4 @@
   <xacro:include filename="$(find so101_description)/urdf/so101_left_arm_camera.urdf.fragment"/>
   <xacro:include filename="$(find so101_description)/urdf/so101_right_arm_camera.urdf.fragment"/>
-  <!-- Modular assembly-task object macros (only plug + socket used here) -->
-  <xacro:include filename="$(find so101_description)/urdf/assembly_objects.urdf.xacro"/>
   <!-- ================= TABLE (industrial aluminum-extrusion bench) ================= -->
   <!-- x = long side = 100 cm -->
@@ -40,6 +38,6 @@
   <!-- ================= ROBOTS =================== -->
   <xacro:property name="robot_y"       value="${table_y/2}"/>
-  <xacro:property name="robot_left_x"  value="-0.25"/>
-  <xacro:property name="robot_right_x" value="0.25"/>
+  <xacro:property name="robot_left_x"  value="-0.15"/>
+  <xacro:property name="robot_right_x" value="0.15"/>
   <xacro:property name="robot_yaw"     value="${-pi/2}"/>
   <!-- ================= OVERHEAD CAMERA GANTRY ================= -->
@@ -51,15 +49,18 @@
   <xacro:property name="cam_yaw"   value="${-pi/2}"/>
   <!-- ================= ASSEMBLY AREA ================= -->
-  <!-- Socket is static, fixed to the table. The plug is a separately
-       spawned free body (models/plug.sdf), not part of this URDF, see
-       workcell_gazebo.launch.py. plug_x/plug_y are kept here only so the
-       launch file's spawn position (world frame: x=plug_x, y=plug_y,
+  <!-- Both the socket (models/socket.sdf, static) and the plug
+       (models/plug.sdf, free body) are spawned separately in
+       workcell_gazebo.launch.py, not part of this URDF, so the socket's
+       position can be changed by editing the launch file's spawn args,
+       without a xacro edit or colcon rebuild, while experimenting.
+       socket_x/socket_y/plug_x/plug_y are kept here only as documentation:
+       the launch file's spawn position (world frame: x=*_x, y=*_y,
        z=table_top_z, since table_link has no rotation/xy-offset from
-       world) stays next to the property that defines it, for the same
-       spot the plug used to occupy when it was welded to the table. -->
+       world) stays next to the property that used to define it, for the
+       same spot each used to occupy when welded to the table. -->
   <xacro:property name="socket_x" value="0.0"/>
-  <xacro:property name="socket_y" value="0.08"/>
-  <xacro:property name="plug_x"   value="0.0"/>
-  <xacro:property name="plug_y"   value="0.16"/>
+  <xacro:property name="socket_y" value="0.10"/>
+  <xacro:property name="plug_x"   value="-0.23"/>
+  <xacro:property name="plug_y"   value="0.08"/>
   <!-- ================= MATERIALS ================= -->
   <material name="bench_top_dark">
@@ -289,11 +290,4 @@
     <origin xyz="0 0 0" rpy="${-pi/2} 0 ${-pi/2}"/>
   </joint>
-  <!-- ================= SOCKET (static) ================= -->
-  <!-- The plug is NOT instantiated here: it's a free rigid body, spawned
-       separately as models/plug.sdf via `ros2 run ros_gz_sim create` in
-       workcell_gazebo.launch.py (at plug_x/plug_y, same spot as before) so
-       it's actually pickable rather than welded to the table. -->
-  <xacro:socket name="socket" parent="table_link"
-    xyz="${socket_x} ${socket_y} 0" rpy="0 0 0"/>
   <!-- ================= ROS2_CONTROL ================ -->
   <xacro:macro name="position_joint" params="name">

File: src/so101_description/urdf/dual_arm_workcell_peghole_gazebo.urdf.xacro (robot description, xacro)
@@ -21,6 +21,4 @@
   <xacro:include filename="$(find so101_description)/urdf/so101_left_arm_camera.urdf.fragment"/>
   <xacro:include filename="$(find so101_description)/urdf/so101_right_arm_camera.urdf.fragment"/>
-  <!-- Modular assembly-task object macros (peg, base plate w/ hole, fixture, tray) -->
-  <xacro:include filename="$(find so101_description)/urdf/assembly_objects.urdf.xacro"/>
   <!-- ================= TABLE (industrial aluminum-extrusion bench) ================= -->
   <!-- x = long side = 100 cm -->
@@ -287,28 +285,21 @@
     <origin xyz="0 0 0" rpy="${-pi/2} 0 ${-pi/2}"/>
   </joint>
-  <!-- ================= ASSEMBLY FIXTURE + BASE PLATE (static) ================= -->
-  <!-- The peg is NOT instantiated here: it's a free rigid body, spawned
-       separately as models/peg.sdf via `ros2 run ros_gz_sim create` in
-       workcell_peghole_gazebo.launch.py (at the same spot it used to
-       occupy: x = fixture_x + 0.09, y = fixture_y) so it's actually
-       pickable rather than welded to the table. -->
-  <xacro:assembly_fixture name="assembly_fixture" parent="table_link"
-    xyz="${fixture_x} ${fixture_y} 0" rpy="0 0 0"/>
-  <xacro:base_plate_with_hole name="base_plate" parent="assembly_fixture_link"
-    xyz="0 0 0.006" rpy="0 0 0"/>
-  <!-- ================= PARTS TRAY ================= -->
-  <!-- Spare pegs stay fixed/decorative: only the functional peg and plug
-       were asked to become pickable, not every loose part in the scene. -->
-  <xacro:parts_tray name="parts_tray" parent="table_link"
-    xyz="${tray_x} ${tray_y} 0" rpy="0 0 0"/>
-  <xacro:peg name="spare_peg_1" parent="parts_tray_link"
-    xyz="-0.03 0.02 0.013" rpy="0 ${pi/2} 0" radius="0.007" length="0.035"/>
-  <xacro:peg name="spare_peg_2" parent="parts_tray_link"
-    xyz="0.02 -0.015 0.013" rpy="0 ${pi/2} ${pi/4}" radius="0.007" length="0.035"/>
-  <!-- ================= SOCKET (static) ================= -->
-  <!-- The plug is likewise spawned separately as models/plug.sdf, not
-       instantiated here, see workcell_peghole_gazebo.launch.py. -->
-  <xacro:socket name="socket" parent="table_link"
-    xyz="${socket_x} ${socket_y} 0" rpy="0 0 0"/>
+  <!-- ================= ASSEMBLY OBJECTS ================= -->
+  <!-- None of assembly_fixture, base_plate, parts_tray, spare_peg_1,
+       spare_peg_2, socket, peg or plug are instantiated here anymore;
+       all are spawned separately as their own SDF models (models/*.sdf)
+       via `ros2 run ros_gz_sim create` in workcell_peghole_gazebo.launch
+       .py instead of being welded into this URDF, so any of them can be
+       repositioned by editing that launch file's spawn args, with no
+       xacro edit or colcon rebuild needed. See that launch file for each
+       one's current world-frame spawn pose (computed from
+       fixture_x/fixture_y/tray_x/tray_y/socket_x/socket_y/plug_x/plug_y
+       above, which are kept here only as documentation of where each
+       used to be welded). peg and plug are free rigid bodies (pickable);
+       assembly_fixture, base_plate, parts_tray, spare_peg_1, spare_peg_2
+       and socket are spawned `<static>true</static>` (fixtures, not
+       pickable parts; spare pegs stay fixed/decorative by original
+       design: only the functional peg and plug were asked to be
+       pickable, not every loose part in the scene). -->
   <!-- ================= ROS2_CONTROL ================ -->
   <xacro:macro name="position_joint" params="name">
